Commit message: Audit of phases 0-6: safety and correctness fixes, end-to-end simulation
An audit (four independent reviews plus end-to-end runs of the real Nav2
stack against a kinematic stand-in) found and fixed:

Safety
- velocity gate: NaN commands became full speed; enable, recovery and
  phone liveness latched forever (they now expire after 1.5 s and the
  mission re-sends at 2 Hz); direction reversal skipped the ramp
- trip: resuming ignored pause, follow-loss and lost localization; one
  _resume() path now checks all three before any Nav2 goal
- elevator creep could not be paused or cancelled
- phone IMU node died on one malformed POST; rosbridge accepted any
  topic from the WiFi (now restricted to the app's own topics)
- firmware parsed the tail of an overlong line as a command

Correctness
- base_link on the floor (ground projections were 8 cm high)
- localization mode, route and outdoor flag latched so late nodes get them;
  map loads retried until map_server answers
- phone clock offset, camera yaw sign, PaddleOCR pinned to 2.x API,
  voice history poisoned by truncated tool calls, phone app stuck after
  a trip, heartbeat timeout, BLE silence, push-to-talk playback

Found by simulation
- door/elevator nodes now 0.8 m from walls so Nav2 can reach them
- sparse Nav2 waypoints (junctions and turns) instead of every 5 m node
- skeleton at the grid's 5 cm resolution, and every graph edge checked
  against the Nav2 grid for the car's width (14 edges through thin GIS
  walls removed); doorways carved into the grids
- elevator exit turns round and drives out forwards

Simulated trips arrive: AQ 3046 (4 of 5 runs), AQ 3150 (spec exit route,
275 m), AQ 6106 (elevator to AQ-06 and two doors). New sim_trip tool
reproduces them. Report: docs/superpowers/audits/2026-10-03-software-audit.md

Co-Authored-By: Claude Opus 5.5 <noreply@anthropic.com>
Claude-Session: https://claude.ai/code/session_015rcd5qBkZsGevG9pressoR

File: ros2_ws/src/guide_bringup/urdf/guide_car.urdf.xacro (robot description, xacro)
@@ -1,4 +1,7 @@
 <?xml version="1.0"?>
-<!-- SFU guide car. Measure the mounts on the built chassis and update the numbers. -->
+<!-- SFU guide car. Measure the mounts on the built chassis and update the numbers.
+     base_link lies on the floor (z = 0 at ground level, between the drive wheels):
+     the perception nodes intersect camera rays with z = 0 in base_link, and the
+     costmap height filters are heights above the floor. -->
 <robot name="guide_car" xmlns:xacro="http://www.ros.org/wiki/xacro">
   <xacro:property name="base_length" value="0.45"/>
@@ -8,5 +11,5 @@
   <!-- Stereo pair: 10 to 15 cm baseline, level, facing forward (spec section 3). -->
   <xacro:property name="cam_x" value="0.20"/>
-  <xacro:property name="cam_z" value="0.45"/>
+  <xacro:property name="cam_z" value="0.45"/>       <!-- lens height above the floor -->
   <xacro:property name="cam_pitch" value="0.20"/>   <!-- radians, nose down -->
   <xacro:property name="stereo_baseline" value="0.12"/>
@@ -14,9 +17,9 @@
   <link name="base_link">
     <visual>
-      <origin xyz="0 0 ${base_height/2}"/>
+      <origin xyz="0 0 ${wheel_radius + base_height/2}"/>
       <geometry><box size="${base_length} ${base_width} ${base_height}"/></geometry>
     </visual>
     <collision>
-      <origin xyz="0 0 ${base_height/2}"/>
+      <origin xyz="0 0 ${wheel_radius + base_height/2}"/>
       <geometry><box size="${base_length} ${base_width} ${base_height}"/></geometry>
     </collision>
@@ -24,5 +27,5 @@
   <joint name="base_joint" type="fixed">
     <parent link="base_footprint"/><child link="base_link"/>
-    <origin xyz="0 0 ${wheel_radius}"/>
+    <origin xyz="0 0 0"/>
   </joint>
   <xacro:macro name="camera" params="name x y z pitch yaw">
@@ -47,5 +50,5 @@
   <joint name="phone_joint" type="fixed">
     <parent link="base_link"/><child link="phone_link"/>
-    <origin xyz="0 0 ${base_height + 0.01}"/>
+    <origin xyz="0 0 ${wheel_radius + base_height + 0.01}"/>
   </joint>
   <!-- External GPS antenna on top (spec section 3). -->

Commit message: QA and audit fixes, ponytail simplifications
Safety and correctness (found by the parallel QA and audit passes):
- mission: no crash when a fix arrives without a position; creep counts
  metres and radians, not time; stale "localized" times out; nav failures
  reset per trip
- firmware: separate PWM floors for driving and pivoting; a dead or
  unplugged ultrasonic reports U -1 and the gate fails closed
- velocity gate: the outdoor flag times out like the other flags
- Claude session: one client under concurrent prewarm and ask; cancel the
  future on timeout; voice raises on an error reply
- student tracker: keep the lock, re-lock only near the last distance;
  rear camera rectified
- URDF: drop base_footprint (the EKF is base_link's only parent)
- sim: pulseIn timing, unplug-bumper hook, door resolved by the route graph

Ponytail pass: unused imports and parameters removed, duplicate helpers
replaced by the existing ones.

Co-Authored-By: Claude Opus 5.5 <noreply@anthropic.com>
Claude-Session: https://claude.ai/code/session_015rcd5qBkZsGevG9pressoR

File: ros2_ws/src/guide_bringup/urdf/guide_car.urdf.xacro (robot description, xacro)
@@ -14,5 +14,4 @@
   <xacro:property name="cam_pitch" value="0.20"/>   <!-- radians, nose down -->
   <xacro:property name="stereo_baseline" value="0.12"/>
-  <link name="base_footprint"/>
   <link name="base_link">
     <visual>
@@ -25,8 +24,5 @@
     </collision>
   </link>
-  <joint name="base_joint" type="fixed">
-    <parent link="base_footprint"/><child link="base_link"/>
-    <origin xyz="0 0 0"/>
-  </joint>
+  <!-- No base_footprint: base_link is on the floor already, and the EKF is its only parent. -->
   <xacro:macro name="camera" params="name x y z pitch yaw">
     <link name="${name}_link"/>

Commit message: RC car dimensions: 75 x 41 cm body, 18 cm wheels
Nav2 footprint, URDF body and wheels, cameras near the front edge
(cam_x 0.30), firmware track width 0.34 m (to measure), simulated chassis
and the ultrasonic on the front bumper.

Co-Authored-By: Claude Opus 5.5 <noreply@anthropic.com>
Claude-Session: https://claude.ai/code/session_015rcd5qBkZsGevG9pressoR

File: ros2_ws/src/guide_bringup/urdf/guide_car.urdf.xacro (robot description, xacro)
@@ -5,10 +5,10 @@
      costmap height filters are heights above the floor. -->
 <robot name="guide_car" xmlns:xacro="http://www.ros.org/wiki/xacro">
-  <xacro:property name="base_length" value="0.45"/>
-  <xacro:property name="base_width" value="0.35"/>
+  <xacro:property name="base_length" value="0.75"/>   <!-- RC car body, 75 x 41 cm -->
+  <xacro:property name="base_width" value="0.41"/>
   <xacro:property name="base_height" value="0.15"/>
-  <xacro:property name="wheel_radius" value="0.08"/>
+  <xacro:property name="wheel_radius" value="0.09"/>  <!-- 18 cm wheels -->
   <!-- Stereo pair: 10 to 15 cm baseline, level, facing forward (spec section 3). -->
-  <xacro:property name="cam_x" value="0.20"/>
+  <xacro:property name="cam_x" value="0.30"/>       <!-- near the front edge (0.375) -->
   <xacro:property name="cam_z" value="0.45"/>       <!-- lens height above the floor -->
   <xacro:property name="cam_pitch" value="0.20"/>   <!-- radians, nose down -->

Commit message: Stereo: 10 cm baseline and a 128-disparity search
With the 50 deg webcams (fx about 690 px at 640 x 360), 12 cm and 64
disparities left everything nearer than 1.3 m out of the stereo depth.
10 cm and 128: from 0.54 m, about 6 cm of depth error at 4 m.

Co-Authored-By: Claude Opus 5.5 <noreply@anthropic.com>
Claude-Session: https://claude.ai/code/session_015rcd5qBkZsGevG9pressoR

File: ros2_ws/src/guide_bringup/urdf/guide_car.urdf.xacro (robot description, xacro)
@@ -9,9 +9,10 @@
   <xacro:property name="base_height" value="0.15"/>
   <xacro:property name="wheel_radius" value="0.09"/>  <!-- 18 cm wheels -->
-  <!-- Stereo pair: 10 to 15 cm baseline, level, facing forward (spec section 3). -->
+  <!-- Stereo pair: 10 cm apart (lens centres), level, facing forward. With the 50 deg
+       webcams and a 128-disparity search, stereo sees from 0.54 m out (spec section 3). -->
   <xacro:property name="cam_x" value="0.30"/>       <!-- near the front edge (0.375) -->
   <xacro:property name="cam_z" value="0.45"/>       <!-- lens height above the floor -->
   <xacro:property name="cam_pitch" value="0.20"/>   <!-- radians, nose down -->
-  <xacro:property name="stereo_baseline" value="0.12"/>
+  <xacro:property name="stereo_baseline" value="0.10"/>
   <link name="base_link">
     <visual>

Commit message: Audit for the real RC car: electrical guards, trim cap, footprint on the rear axle, robust voice and perception startup
Drive path: the ESP32 firmware refuses to run if a measured controller voltage
is above 3.3 V, maps each end of travel separately, drops pinMode on DAC pins;
the bridge opens the port with DTR/RTS low (asserting them resets the board
and leaves the controller inputs floating). Speed trim capped at 0.12 m/s or
60 % of the speed asked; the gate's reverse tick sends no turn.

Navigation: footprint about the rear axle (0.63 m ahead, 0.12 m behind) with
the camera and bumper mounts moved; progress checker allows 60 s (the gate
holds the car for people); wall-snap at most once per 10 s. Gyro bias learns
only from fresh, non-null odometry in its own time base and a nearly-still gyro.

Voice and perception: the voice node survives a missing Gemini key or
microphone and warns on a missing ElevenLabs key; TTS as PCM wrapped locally;
Gemini model pinned; a missing model file is a clear fatal; an uncalibrated
camera keeps the safe any-person-is-close path; RTAB-Map localization refuses
to start without the floor's database. iOS Sensor Logger accelerometer and
gravity paired by time. Ports from /dev/serial/by-id (ESP32 is ttyUSB0).

Docs: the RC car runbook (wiring, measuring, flashing, bench test,
calibration, first drive, the phone), spec section 10 and the stale
tank-steering text; audit doc third pass.

Co-Authored-By: Claude Fable 5.1 <noreply@anthropic.com>
Claude-Session: https://claude.ai/code/session_015rcd5qBkZsGevG9pressoR

File: ros2_ws/src/guide_bringup/urdf/guide_car.urdf.xacro (robot description, xacro)
@@ -1,9 +1,12 @@
 <?xml version="1.0"?>
-<!-- SFU guide car. Measure the mounts on the built chassis and update the numbers.
-     base_link lies on the floor (z = 0 at ground level, between the drive wheels):
+<!-- SFU guide car: a stock RC car, Ackermann steering. Measure the mounts on the built
+     chassis and update the numbers. base_link lies on the floor (z = 0 at ground level)
+     at the centre of the REAR axle, which the bicycle model turns about; the 75 cm body
+     reaches rear_overhang behind it and the rest ahead (match nav2.yaml's footprint):
      the perception nodes intersect camera rays with z = 0 in base_link, and the
      costmap height filters are heights above the floor. -->
 <robot name="guide_car" xmlns:xacro="http://www.ros.org/wiki/xacro">
   <xacro:property name="base_length" value="0.75"/>   <!-- RC car body, 75 x 41 cm -->
+  <xacro:property name="rear_overhang" value="0.12"/> <!-- rear axle to the back of the body: measure -->
   <xacro:property name="base_width" value="0.41"/>
   <xacro:property name="base_height" value="0.15"/>
@@ -11,5 +14,5 @@
   <!-- Stereo pair: 10 cm apart (lens centres), level, facing forward. With the 50 deg
        webcams and a 128-disparity search, stereo sees from 0.54 m out (spec section 3). -->
-  <xacro:property name="cam_x" value="0.30"/>       <!-- near the front edge (0.375) -->
+  <xacro:property name="cam_x" value="0.50"/>       <!-- ahead of the rear axle; the body ends at 0.63 -->
   <xacro:property name="cam_z" value="0.45"/>       <!-- lens height above the floor -->
   <xacro:property name="cam_pitch" value="0.20"/>   <!-- radians, nose down -->
@@ -17,9 +20,9 @@
   <link name="base_link">
     <visual>
-      <origin xyz="0 0 ${wheel_radius + base_height/2}"/>
+      <origin xyz="${base_length/2 - rear_overhang} 0 ${wheel_radius + base_height/2}"/>
       <geometry><box size="${base_length} ${base_width} ${base_height}"/></geometry>
     </visual>
     <collision>
-      <origin xyz="0 0 ${wheel_radius + base_height/2}"/>
+      <origin xyz="${base_length/2 - rear_overhang} 0 ${wheel_radius + base_height/2}"/>
       <geometry><box size="${base_length} ${base_width} ${base_height}"/></geometry>
     </collision>
@@ -45,5 +48,5 @@
   <xacro:camera name="iphone_camera" x="${cam_x}" y="0" z="${cam_z}" pitch="${cam_pitch}" yaw="0"/>
   <!-- Phase 6 rear camera, facing backwards (with cameras:=iphone, the webcam). -->
-  <xacro:camera name="rear_camera" x="${-base_length/2}" y="0" z="${cam_z}" pitch="0.1" yaw="${pi}"/>
+  <xacro:camera name="rear_camera" x="${-rear_overhang}" y="0" z="${cam_z}" pitch="0.1" yaw="${pi}"/>
   <!-- Phone lying flat, screen up, top edge forward (spec section 3). -->
   <link name="phone_link"/>

Commit message: Cameras at 28 cm, 5 degrees up, the 1080p pair's 70 degree view
Co-Authored-By: Claude Fable 5.1 <noreply@anthropic.com>
Claude-Session: https://claude.ai/code/session_015rcd5qBkZsGevG9pressoR

File: ros2_ws/src/guide_bringup/urdf/guide_car.urdf.xacro (robot description, xacro)
@@ -15,6 +15,9 @@
        webcams and a 128-disparity search, stereo sees from 0.54 m out (spec section 3). -->
   <xacro:property name="cam_x" value="0.50"/>       <!-- ahead of the rear axle; the body ends at 0.63 -->
-  <xacro:property name="cam_z" value="0.45"/>       <!-- lens height above the floor -->
-  <xacro:property name="cam_pitch" value="0.20"/>   <!-- radians, nose down -->
+  <xacro:property name="cam_z" value="0.28"/>       <!-- lens height above the floor (the RC car's mount) -->
+  <!-- 5 deg nose UP (negative pitch): from 28 cm, level would see nothing above 1.1 m at 2 m; tilted up
+       the pair sees to 1.3 m at 2 m and 1.8 m at 3 m (door signs from about 2 m, with capture:=720p)
+       and the floor from 0.95 m ahead (the bumper covers nearer). -->
+  <xacro:property name="cam_pitch" value="-0.09"/>
   <xacro:property name="stereo_baseline" value="0.10"/>
   <link name="base_link">
